File: PCB_LABORDE-TASTET.kicad_pcb (KiCad board)
At the start: 2 copper layers, 116.8 x 97.8 mm, 51 parts, among them J2 Conn_01x02, J3 Conn_01x03, Q1 2N2907, Q10 TIP32, Q11 BD138, Q12 TIP31, Q13 2N2222, Q2 2N2907, Q3 2N2907, Q4 2N2222, Q5 2N2222, Q6 2N2907, Q7 2N2907, Q8 BD139, Q9 BD139, U1 Relay_1CT, U2 Jack_Mono

Commit message: AVIS PLACEMENT KICAD VERSION 2 LABORDE-TASTET RAHLI
Parts:
- C1, C3, C4, C6: footprint Capacitor_THT:CP_Radial_D8.0mm_P5.00mm -> importation:CP_Radial_D8.0mm_P5.00mm
- C10, C8: footprint Capacitor_THT:CP_Radial_D12.5mm_P5.00mm -> importation:CP_Radial_D12.5mm_P5.00mm
- C11, C2, C5, C7, C9: footprint Capacitor_THT:C_Rect_L7.2mm_W3.5mm_P5.00mm_FKS2_FKP2_MKS2_MKP2 -> importation:C_Rect_L7.2mm_W3.5mm_P5.00mm_FKS2_FKP2_MKS2_MKP2
- D1, D2, Dz1: footprint Diode_THT:D_DO-35_SOD27_P10.16mm_Horizontal -> importation:D_DO-35_SOD27_P10.16mm_Horizontal
- H51, HS2: footprint Heatsink:Heatsink_Fischer_SK104-STC-STIC_35x13mm_2xDrill2.5mm -> importation:Heatsink_Fischer_SK104-STC-STIC_35x13mm_2xDrill2.5mm
- J2: footprint Connector_Phoenix_MSTB:PhoenixContact_MSTBVA_2,5_2-G-5,08_1x02_P5.08mm_Vertical -> importation:PhoenixContact_MSTBVA_2,5_2-G-5,08_1x02_P5.08mm_Vertical
- J3: footprint Connector_Phoenix_MSTB:PhoenixContact_MSTBVA_2,5_3-G-5,08_1x03_P5.08mm_Vertical -> importation:PhoenixContact_MSTBVA_2,5_3-G-5,08_1x03_P5.08mm_Vertical
- Q1, Q13, Q2, Q3, Q4, Q5, Q6, Q7: footprint Package_TO_SOT_THT:TO-18-3 -> importation:TO-18-3
- Q10, Q12: footprint Package_TO_SOT_THT:TO-220-3_Vertical -> importation:TO-220-3_Vertical
- Q11, Q8, Q9: footprint Package_TO_SOT_THT:TO-126-3_Vertical -> importation:TO-126-3_Vertical
- R1, R10, R13, R14, R15, R16, R2, R3, R4, R5, R6, R7, R8, R9: footprint Resistor_THT:R_Axial_DIN0207_L6.3mm_D2.5mm_P10.16mm_Horizontal -> importation:R_Axial_DIN0207_L6.3mm_D2.5mm_P10.16mm_Horizontal
- R11, R12: footprint Resistor_THT:R_Axial_DIN0516_L15.5mm_D5.0mm_P20.32mm_Horizontal -> importation:R_Axial_DIN0516_L15.5mm_D5.0mm_P20.32mm_Horizontal
- moved Q12 4.37 mm to (181.5, 77.0)
- moved H51 4.10 mm to (108.2, 77.8)
- moved Q10 3.06 mm to (106.0, 81.9)
- moved C5 2.95 mm to (108.5, 50.0)
- moved C7 2.79 mm to (119.2, 50.0)
- moved HS2 1.89 mm to (179.0, 74.5)
- moved C6 1.67 mm to (125.8, 40.0)
- moved Q13 1.58 mm to (129.4, 50.0)
- moved C3 1.57 mm to (164.2, 44.3)
- moved C8 1.47 mm to (118.4, 63.1)
- moved J2 1.26 mm to (184.4, 39.6)
- moved J3 1.23 mm to (118.0, 39.5)
- moved U2 0.52 mm to (132.5, 132.3)
Connections:
- J2 pad 1: /HP -> GND
- J2 pad 2: GND -> /HP

Commit message: AVIS PLACEMENT KICAD VERSION 4 LABORDE-TASTET RAHLI
Parts:
- moved Q4 28.6 mm to (148.2, 103.8)
- moved C2 23.3 mm to (161.4, 104.0)
- moved Q12 10.6 mm to (182.3, 66.5)
- moved C11 8.47 mm to (178.8, 57.5), turned to 180 degrees
- moved R4 6.34 mm to (134.0, 112.5)
- moved C10 4.56 mm to (188.5, 52.7)
- moved HS2 3.71 mm to (179.2, 70.8)
- moved R5 2.70 mm to (163.3, 119.8)
- moved Q5 2.56 mm to (183.1, 90.0), turned to 180 degrees
- moved R9 2.23 mm to (94.0, 103.1)
- moved R7 2.15 mm to (93.9, 96.8)
- moved R6 2.10 mm to (190.0, 92.9)
- moved RV2 1.82 mm to (127.0, 111.5)
- moved R14 1.41 mm to (194.5, 94.2)
- moved U2 1.00 mm to (133.5, 132.3)
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Routing:
- net +12V: track 0.00 -> 228.9 mm
- net -12V: track 0.00 -> 207.4 mm
- net Net-(R11-Pad2): track 0.00 -> 87.5 mm, vias 0 -> 2
- net Net-(C2-Pad1): track 0.00 -> 79.7 mm
- net Net-(Q2-Pad2): track 0.00 -> 50.6 mm
- net /HP: track 0.00 -> 48.1 mm
- net Net-(Q4-Pad1): track 0.00 -> 45.0 mm
- net Net-(C2-Pad2): track 0.00 -> 40.4 mm
- net Net-(Q10-Pad2): track 0.00 -> 39.4 mm
- net Net-(Q11-Pad1): track 0.00 -> 35.1 mm
- net Net-(Q6-Pad3): track 0.00 -> 34.1 mm
- net Net-(Q11-Pad2): track 0.00 -> 30.4 mm
- net Net-(C1-Pad2): track 0.00 -> 26.2 mm
- net Net-(Q6-Pad2): track 0.00 -> 22.9 mm
- net Net-(C1-Pad1): track 0.00 -> 22.4 mm, vias 0 -> 2
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- added copper zone on B.Cu, net GND
- added copper zone on F.Cu, net GND
Other:
- board text added: "Bottom"
- board text added: "Laborde-Tastet Antonin Rahli Oussama"
- board text added: "Top"

Commit message: AVIS ROUTAGE KICAD VERSION 5 LABORDE-TASTET RAHLI
Routing:
- net Net-(C1-Pad1): track 22.4 -> 23.4 mm
Changed lines of the file:
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@@
     (date "2022-04-02")
     (company "3 IMACS Groupe E")
-    (comment 1 "Version 4")
-    (comment 2 "Retrait d' 1 des 3 straps,  branchement du + 12V entre C9 et C4")
-    (comment 3 "plan de masse  + nom en couche Bottom")
+    (comment 1 "Version 5")
+    (comment 2 "strap en horizontal au lieux de diagonal")
+    (comment 3 "Pistes élargies")
     (comment 4 "Modifs:")
   )
@@
     (effects (font (size 1.5 1.5) (thickness 0.3)) (justify mirror))
   )
-  (via (at 171.75 112.25) (size 1.9) (drill 0.6) (layers "F.Cu" "B.Cu") (net 1))
-  (via (at 169.25 114.75) (size 1.9) (drill 0.6) (layers "F.Cu" "B.Cu") (net 1))
-  (segment (start 169.25 114.75) (end 169.5 114.5) (width 0.6) (layer "B.Cu") (net 1))
+  (via (at 171.625 112.375) (size 1.9) (drill 0.6) (layers "F.Cu" "B.Cu") (net 1))
+  (via (at 167.3 112.65) (size 1.9) (drill 0.6) (layers "F.Cu" "B.Cu") (net 1))
+  (segment (start 167.05 112.9) (end 167.225 112.725) (width 0.6) (layer "B.Cu") (net 1))
   (segment (start 162.670195 124.549805) (end 157.77785 124.549805) (width 0.6) (layer "B.Cu") (net 1))
-  (segment (start 173.01785 110.98215) (end 171.75 112.25) (width 0.6) (layer "B.Cu") (net 1))
-  (segment (start 169.25 114.75) (end 167.05 116.95) (width 0.6) (layer "B.Cu") (net 1))
+  (segment (start 171.625 112.375) (end 171.5 112.5) (width 0.6) (layer "B.Cu") (net 1))
+  (segment (start 167.05 114.65) (end 167.05 112.9) (width 0.6) (layer "B.Cu") (net 1))
+  (segment (start 167.05 116.95) (end 167.05 114.65) (width 0.6) (layer "B.Cu") (net 1))
+  (segment (start 173.01785 110.98215) (end 171.625 112.375) (width 0.6) (layer "B.Cu") (net 1))
+  (segment (start 167.225 112.725) (end 167.3 112.65) (width 0.6) (layer "B.Cu") (net 1))
   (segment (start 173.01785 108.537456) (end 173.01785 110.98215) (width 0.6) (layer "B.Cu") (net 1))
-  (segment (start 171.75 112.25) (end 171.5 112.5) (width 0.6) (layer "B.Cu") (net 1))
+  (segment (start 167.3 112.65) (end 167.4 112.55) (width 0.6) (layer "B.Cu") (net 1))
   (segment (start 167.05 120.17) (end 162.670195 124.549805) (width 0.6) (layer "B.Cu") (net 1))
   (segment (start 167.05 116.95) (end 167.05 120.17) (width 0.6) (layer "B.Cu") (net 1))
@@
   (segment (start 155.87285 112.347456) (end 161.58785 112.347456) (width 0.6) (layer "B.Cu") (net 11))
   (segment (start 161.58785 118.05785) (end 163.33 119.8) (width 0.6) (layer "B.Cu") (net 11))
-  (segment (start 179.05 39.6675) (end 179.05 46.95) (width 0.6) (layer "B.Cu") (net 12))
-  (segment (start 179.05 46.95) (end 155.5175 70.4825) (width 0.6) (layer "B.Cu") (net 12))
-  (segment (start 155.5175 70.4825) (end 147.9875 70.4825) (width 0.6) (layer "B.Cu") (net 12))
+  (segment (start 179.05 39.6675) (end 179.05 46.95) (width 1.1) (layer "B.Cu") (net 12))
+  (segment (start 179.05 46.95) (end 155.5175 70.4825) (width 1.1) (layer "B.Cu") (net 12))
+  (segment (start 155.5175 70.4825) (end 147.9875 70.4825) (width 1.1) (layer "B.Cu") (net 12))
   (segment (start 171.11285 114.152456) (end 167.30285 110.342456) (width 0.6) (layer "B.Cu") (net 13))
   (segment (start 171.11285 117.962456) (end 171.11285 114.152456) (width 0.6) (layer "B.Cu") (net 13))
@@
   (segment (start 121.39 97.269022) (end 125.985978 101.865) (width 0.6) (layer "B.Cu") (net 23))
   (segment (start 121.39 96.81) (end 121.39 97.269022) (width 0.6) (layer "B.Cu") (net 23))
-  (segment (start 115.85 89.43) (end 121.07 89.43) (width 0.6) (layer "B.Cu") (net 24))
+  (segment (start 115.85 89.43) (end 121.07 89.43) (width 1.1) (layer "B.Cu") (net 24))
   (segment (start 110.105 85.5) (end 113.5 85.5) (width 0.6) (layer "B.Cu") (net 24))
-  (segment (start 121.07 89.43) (end 132.15 78.35) (width 0.6) (layer "B.Cu") (net 24))
+  (segment (start 121.07 89.43) (end 132.15 78.35) (width 1.1) (layer "B.Cu") (net 24))
   (segment (start 115.85 87.85) (end 115.85 89.43) (width 0.6) (layer "B.Cu") (net 24))
   (segment (start 108.5 83.895) (end 110.105 85.5) (width 0.6) (layer "B.Cu") (net 24))
   (segment (start 108.5 81.945) (end 108.5 83.895) (width 0.6) (layer "B.Cu") (net 24))
   (segment (start 113.5 85.5) (end 115.85 87.85) (width 0.6) (layer "B.Cu") (net 24))
-  (segment (start 132.15 78.35) (end 132.15 72.4) (width 0.6) (layer "B.Cu") (net 24))
+  (segment (start 132.15 78.35) (end 132.15 72.4) (width 1.1) (layer "B.Cu") (net 24))
   (segment (start 112.5 87) (end 113.31 87.81) (width 0.6) (layer "B.Cu") (net 25))
   (segment (start 105.96 83.895) (end 109.065 87) (width 0.6) (layer "B.Cu") (net 25))
@@
   (segment (start 180 80.5) (end 179.5 80.5) (width 0.6) (layer "B.Cu") (net 30))
   (segment (start 185.5 80.5) (end 180 80.5) (width 0.6) (layer "B.Cu") (net 30))
-  (segment (start 151.71 89.79) (end 161 80.5) (width 0.6) (layer "B.Cu") (net 30))
+  (segment (start 151.71 89.79) (end 161 80.5) (width 1.1) (layer "B.Cu") (net 30))
   (segment (start 132.15 92.72) (end 138.04 92.72) (width 0.6) (layer "B.Cu") (net 30))
-  (segment (start 140.3675 67.9425) (end 138 70.31) (width 0.6) (layer "B.Cu") (net 30))
+  (segment (start 140.3675 67.9425) (end 138 70.31) (width 1.1) (layer "B.Cu") (net 30))
   (segment (start 140.19 89.01) (end 140.97 89.79) (width 0.6) (layer "B.Cu") (net 30))
-  (segment (start 138 75.46) (end 140.19 77.65) (width 0.6) (layer "B.Cu") (net 30))
-  (segment (start 140.97 89.79) (end 151.71 89.79) (width 0.6) (layer "B.Cu") (net 30))
+  (segment (start 138 75.46) (end 140.19 77.65) (width 1.1) (layer "B.Cu") (net 30))
+  (segment (start 140.97 89.79) (end 151.71 89.79) (width 1.1) (layer "B.Cu") (net 30))
   (segment (start 138.04 92.72) (end 140.97 89.79) (width 0.6) (layer "B.Cu") (net 30))
-  (segment (start 161 80.5) (end 173.5 80.5) (width 0.6) (layer "B.Cu") (net 30))
-  (segment (start 140.19 77.65) (end 140.19 89.01) (width 0.6) (layer "B.Cu") (net 30))
+  (segment (start 161 80.5) (end 173.5 80.5) (width 1.1) (layer "B.Cu") (net 30))
+  (segment (start 140.19 77.65) (end 140.19 89.01) (width 1.1) (layer "B.Cu") (net 30))
   (segment (start 194.5 84.085) (end 189.085 84.085) (width 0.6) (layer "B.Cu") (net 30))
   (segment (start 173.5 80.5) (end 174 80.5) (width 0.6) (layer "B.Cu") (net 30))
-  (segment (start 138 70.31) (end 138 75.46) (width 0.6) (layer "B.Cu") (net 30))
+  (segment (start 138 70.31) (end 138 75.46) (width 1.1) (layer "B.Cu") (net 30))
   (zone (net 6) (net_name "GND") (layer "F.Cu") (hatch edge 0.508)
     (connect_pads (clearance 0.508))
