File: PCB_LABORDE-TASTET.kicad_sch (KiCad schematic)
At the start: 51 parts, among them J2 Conn_01x02, J3 Conn_01x03, Q1 2N2907, Q10 TIP32, Q11 BD138, Q12 TIP31, Q13 2N2222, Q2 2N2907, Q3 2N2907, Q4 2N2222, Q5 2N2222, Q6 2N2907, Q7 2N2907, Q8 BD139, Q9 BD139, U1 Relay_1CT, U2 Jack_Mono

Commit message: AVIS PLACEMENT KICAD VERSION 2 LABORDE-TASTET RAHLI
Parts:
- C1, C3, C4, C6: footprint Capacitor_THT:CP_Radial_D8.0mm_P5.00mm -> (none)
- C10, C8: footprint Capacitor_THT:CP_Radial_D12.5mm_P5.00mm -> (none)
- C11, C2, C5, C7, C9: footprint Capacitor_THT:C_Rect_L7.2mm_W3.5mm_P5.00mm_FKS2_FKP2_MKS2_MKP2 -> (none)
- D1, D2, Dz1: footprint Diode_THT:D_DO-35_SOD27_P10.16mm_Horizontal -> (none)
- H51, HS2: footprint Heatsink:Heatsink_Fischer_SK104-STC-STIC_35x13mm_2xDrill2.5mm -> (none)
- J2: footprint Connector_Phoenix_MSTB:PhoenixContact_MSTBVA_2,5_2-G-5,08_1x02_P5.08mm_Vertical -> (none)
- J3: footprint Connector_Phoenix_MSTB:PhoenixContact_MSTBVA_2,5_3-G-5,08_1x03_P5.08mm_Vertical -> (none)
- Q1, Q13, Q2, Q3, Q4, Q5, Q6, Q7: footprint Package_TO_SOT_THT:TO-18-3 -> (none)
- Q10, Q12: footprint Package_TO_SOT_THT:TO-220-3_Vertical -> (none)
- Q11, Q8, Q9: footprint Package_TO_SOT_THT:TO-126-3_Vertical -> (none)
- R1, R15: footprint Resistor_THT:R_Axial_DIN0207_L6.3mm_D2.5mm_P10.16mm_Horizontal -> importation:R_Axial_DIN0207_L6.3mm_D2.5mm_P10.16mm_Horizontal
- R10, R13, R14, R16, R2, R3, R4, R5, R6, R7, R8, R9: footprint Resistor_THT:R_Axial_DIN0207_L6.3mm_D2.5mm_P10.16mm_Horizontal -> (none)
- R12: value (none) -> R
Connections:
- net GND: now also J2.1 (Pin_1); no longer J2.2 (Pin_2)
- net HP: now also J2.2 (Pin_2); no longer J2.1 (Pin_1)

Commit message: AVIS PLACEMENT KICAD VERSION 4 LABORDE-TASTET RAHLI
Parts:
- C1, C3, C4, C6: footprint (none) -> importation:CP_Radial_D8.0mm_P5.00mm
- C10, C8: footprint (none) -> importation:CP_Radial_D12.5mm_P5.00mm
- C11, C2, C5, C7, C9: footprint (none) -> importation:C_Rect_L7.2mm_W3.5mm_P5.00mm_FKS2_FKP2_MKS2_MKP2
- D1, D2, Dz1: footprint (none) -> importation:D_DO-35_SOD27_P10.16mm_Horizontal
- H51, HS2: footprint (none) -> importation:Heatsink_Fischer_SK104-STC-STIC_35x13mm_2xDrill2.5mm
- J2: footprint (none) -> importation:PhoenixContact_MSTBVA_2,5_2-G-5,08_1x02_P5.08mm_Vertical
- J3: footprint (none) -> importation:PhoenixContact_MSTBVA_2,5_3-G-5,08_1x03_P5.08mm_Vertical
- Q1, Q13, Q2, Q3, Q4, Q5, Q6, Q7: footprint (none) -> importation:TO-18-3
- Q10, Q12: footprint (none) -> importation:TO-220-3_Vertical
- Q11, Q8, Q9: footprint (none) -> importation:TO-126-3_Vertical
- R10, R13, R14, R16, R2, R3, R4, R5, R6, R7, R8, R9: footprint (none) -> importation:R_Axial_DIN0207_L6.3mm_D2.5mm_P10.16mm_Horizontal
- R11, R12: footprint (none) -> importation:R_Axial_DIN0516_L15.5mm_D5.0mm_P20.32mm_Horizontal
Other:
- title: Schéma Ampli Audio Laborde-Tastet / Rhali -> Schéma Ampli Audio Laborde-Tastet / Rahli
